File: beaglemic-cape/beaglemic-cape.sch (KiCad schematic (older format))
At the start: 9 parts, among them J1 USB_OTG, J2 PB_P1, J24 BBAI_FAN, J3 EXT_5V, J4 PB_P2, J5 BBAI_P8, J6 ICE40_EXT, J7 BBAI_P9

Commit message: beaglemic-cape: Shrink PCB to 100x100mm
Let's keep the PCB in the hobby price range.

Version 1.0-rc2

TODO: Route me!

Signed-off-by: Dimitar Dimitrov <dimitar@dinux.eu>
Parts:
- added H1, H2, H3, H4: MountingHole_Pad, MountingHole:MountingHole_3.2mm_M3_ISO14580_Pad, symbol Mechanical:MountingHole_Pad
- renumbered J5 to BBAI_P8, J7 to BBAI_P9, J6 to ICE40HX8K-EVB1, J24 to J4, J2 to PB_P1, J4 to PB_P2
Connections:
- net GND: now also H1.1, H2.1, H3.1, H4.1
Other:
- note added: "WARNING: There is no cutout for the ethernet connector! \nNeed to use extension headers or a suitable additional cape."
- note removed: "WARNING: There is not cutout for the ethernet connector! \nNeed to use extension headers or a suitable additional cape."
- note removed: "iCE40HX8K-EVB"
